Commit message: found original repo i am stupid

File: urdf/robot_pit_end_effector.urdf (robot description, URDF)
Before this commit: robot pit_robot_assembly, 16 links, 15 joints
Links:
- link base_link: geometry collision mesh filename=package://hanford_wire_manipulator_with_camera_description/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; visual mesh filename=package://hanford_wire_manipulator_with_camera_description/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
- link end_effector: geometry collision mesh filename=package://hanford_wire_manipulator_with_camera_description/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 scale=0.001 0.001 0.001; visual mesh filename=package://hanford_wire_manipulator_with_camera_description/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 scale=0.001 0.001 0.001
- link link_1: geometry collision mesh filename=package://hanford_wire_manipulator_with_camera_description/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; visual mesh filename=package://hanford_wire_manipulator_with_camera_description/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
- link link_2: geometry collision mesh filename=package://hanford_wire_manipulator_with_camera_description/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; visual mesh filename=package://hanford_wire_manipulator_with_camera_description/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
- link pit_base_link: geometry collision mesh filename=package://hanford_wire_manipulator_with_camera_description/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; visual mesh filename=package://hanford_wire_manipulator_with_camera_description/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
- link pulley_drive: geometry collision mesh filename=package://hanford_wire_manipulator_with_camera_description/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 scale=0.001 0.001 0.001; visual mesh filename=package://hanford_wire_manipulator_with_camera_description/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 scale=0.001 0.001 0.001
- link zed_x_mini_base: geometry collision mesh filename=package://hanford_wire_manipulator_with_camera_description/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 scale=1. 1. 1.; collision mesh filename=package://hanford_wire_manipulator_with_camera_description/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 scale=1. 1. 1.

Commit message: base link is pipe entry, working again but nothign is moving also i moved files around (mistake)

File: urdf/robot_pit_end_effector.urdf (robot description, URDF)
Before this commit: robot pit_robot_assembly, 16 links, 15 joints
Links:
- removed link pit_base_link
Joints:
- removed joint pit_to_entry
