Commit message: edited urdf to bring back camera link

File: urdf/robot_pit_end_effector_edited.urdf (robot description, URDF)
Before this commit: robot pit_robot_assembly, 14 links, 14 joints
Links:
- added link camera_link
Joints:
- joint camera_link_to_pulley: child zed_x_mini_base -> camera_link
